File: KiCad source/Q17-95x75.kicad_pcb (KiCad board)
At the start: 2 copper layers, 96.5 x 76.2 mm, 84 parts, among them J1 TerminalBlock, Q1 IRF610, Q10 KSA992, Q11 BS250P, Q12 KSC1845, Q13 IRF610, Q14 IRF9610, Q15 FQA46N15, Q16 FQA36P15, Q2 KSA992, Q3 KSC1845, Q4 IRF9610, Q5 IRF9610, Q6 IRF610, Q7 KSC1845, Q8 2N7000, Q9 BS250P, U1 DIP-8_W7.62mm_Socket, U1 OPA1641

Commit message: Update Diagram and PCB to 1.0b13
Other:
- board text added: "Q17 1.0b13"
- board text removed: "Q17 1.0b12"
Changed lines of the file:
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@@
     (title "QUAD405 Reborn")
     (date "2021-11-14")
-    (rev "1.0b12")
+    (rev "1.0b13")
     (company "PCB design by Stef")
     (comment 1 "Zize 95 x 75 mm")
@@
     (effects (font (size 0.5 0.5) (thickness 0.125)))
   )
-  (gr_text "Q17 1.0b12" (at 142.295559 112.014) (layer "F.SilkS")
+  (gr_text "Q17 1.0b13" (at 142.295559 112.014) (layer "F.SilkS")
     (effects (font (size 1 1) (thickness 0.25)))
   )
