File: KiCad source/Q17-Mini.kicad_sch (KiCad schematic)
At the start: 80 parts, among them J1 Input, J2-1 SPK+, J2-2 SPK-, J3-1 V+, J3-2 GND, J3-3 V-, Q1 IRF610, Q10 KSA992, Q11 BS250P, Q12 BD139, Q13 IRF610, Q14 IRF9610, Q15 FQA46N15, Q16 FQA36P15, Q2 KSA992, Q3 KSC1845, Q4 IRF9610, Q5 FQP3P20, Q6 FQP3N30, Q7 KSC1845, Q8 ZVN4206AV, Q9 BS250P, U1 OPA1641

Commit message: Update Q17-Mini.kicad_sch
Other:
- note added: "R27 : Use good low noise and low ppm 1W resistor."
- note removed: "R27 : Vishay Dale 1W (CMF60560R00JKR6) or good low ppm resistor."
- note removed: "Resistors 1W and 2W : Vishay PR01 and PR02 (except R27)."
Changed lines of the file:
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@@
-(kicad_sch (version 20210621) (generator eeschema)
+(kicad_sch (version 20211123) (generator eeschema)
   (paper "A4")
   (title_block
     (title "Q17-Mini Amplifier")
-    (date "2021-11-23")
-    (rev "1.0.7")
+    (date "2021-11-27")
+    (rev "1.0.8")
     (company "by eng. Tiberiu Vicol")
     (comment 1 "Modified by Stef for the Q17-Mini project")
     (comment 4 "Q17 a QUAD405 audiophile approach")
   )
-  (junction (at 194.31 23.876) (diameter 1.016) (color 0 0 0 0))
-  (junction (at 178.816 141.478) (diameter 1.016) (color 0 0 0 0))
-  (junction (at 241.3 141.4597) (diameter 0) (color 0 0 0 0))
-  (junction (at 213.106 141.478) (diameter 1.016) (color 0 0 0 0))
-  (junction (at 49.53 103.124) (diameter 1.016) (color 0 0 0 0))
-  (junction (at 67.818 106.934) (diameter 1.016) (color 0 0 0 0))
-  (junction (at 203.2 130.048) (diameter 1.016) (color 0 0 0 0))
-  (junction (at 178.816 74.93) (diameter 1.016) (color 0 0 0 0))
-  (junction (at 127.762 47.244) (diameter 1.016) (color 0 0 0 0))
-  (junction (at 203.2 35.814) (diameter 1.016) (color 0 0 0 0))
-  (junction (at 84.328 47.498) (diameter 1.016) (color 0 0 0 0))
-  (junction (at 178.816 63.754) (diameter 1.016) (color 0 0 0 0))
-  (junction (at 219.71 95.758) (diameter 1.016) (color 0 0 0 0))
-  (junction (at 78.994 23.876) (diameter 1.016) (color 0 0 0 0))
-  (junction (at 185.42 141.478) (diameter 1.016) (color 0 0 0 0))
-  (junction (at 67.818 64.77) (diameter 1.016) (color 0 0 0 0))
-  (junction (at 194.31 141.478) (diameter 1.016) (color 0 0 0 0))
-  (junction (at 92.71 124.46) (diameter 1.016) (color 0 0 0 0))
-  (junction (at 213.106 23.876) (diameter 1.016) (color 0 0 0 0))
-  (junction (at 79.502 76.454) (diameter 1.016) (color 0 0 0 0))
-  (junction (at 236.982 81.026) (diameter 1.016) (color 0 0 0 0))
-  (junction (at 138.43 39.116) (diameter 1.016) (color 0 0 0 0))
-  (junction (at 78.994 47.498) (diameter 1.016) (color 0 0 0 0))
-  (junction (at 178.816 23.876) (diameter 1.016) (color 0 0 0 0))
-  (junction (at 227.33 81.026) (diameter 1.016) (color 0 0 0 0))
-  (junction (at 219.71 23.876) (diameter 1.016) (color 0 0 0 0))
-  (junction (at 168.402 81.026) (diameter 1.016) (color 0 0 0 0))
-  (junction (at 116.332 58.166) (diameter 1.016) (color 0 0 0 0))
-  (junction (at 92.71 141.478) (diameter 1.016) (color 0 0 0 0))
-  (junction (at 147.32 81.026) (diameter 1.016) (color 0 0 0 0))
-  (junction (at 78.994 117.856) (diameter 1.016) (color 0 0 0 0))
-  (junction (at 240.03 23.9261) (diameter 0) (color 0 0 0 0))
-  (junction (at 78.994 141.478) (diameter 1.016) (color 0 0 0 0))
-  (junction (at 92.71 23.876) (diameter 1.016) (color 0 0 0 0))
-  (junction (at 232.41 141.478) (diameter 1.016) (color 0 0 0 0))
-  (junction (at 219.71 141.478) (diameter 1.016) (color 0 0 0 0))
-  (junction (at 178.816 123.952) (diameter 1.016) (color 0 0 0 0))
-  (junction (at 138.43 55.626) (diameter 1.016) (color 0 0 0 0))
-  (junction (at 67.818 57.15) (diameter 1.016) (color 0 0 0 0))
-  (junction (at 147.32 95.758) (diameter 1.016) (color 0 0 0 0))
-  (junction (at 56.642 83.312) (diameter 1.016) (color 0 0 0 0))
-  (junction (at 42.672 73.914) (diameter 1.016) (color 0 0 0 0))
-  (junction (at 240.03 23.876) (diameter 0) (color 0 0 0 0))
-  (junction (at 92.71 40.894) (diameter 1.016) (color 0 0 0 0))
-  (junction (at 178.816 107.188) (diameter 1.016) (color 0 0 0 0))
-  (junction (at 186.944 23.876) (diameter 1.016) (color 0 0 0 0))
-  (junction (at 138.43 23.876) (diameter 1.016) (color 0 0 0 0))
-  (junction (at 116.332 23.876) (diameter 1.016) (color 0 0 0 0))
-  (junction (at 232.41 23.876) (diameter 1.016) (color 0 0 0 0))
-  (junction (at 92.964 76.454) (diameter 1.016) (color 0 0 0 0))
-  (junction (at 138.43 113.792) (diameter 1.016) (color 0 0 0 0))
-  (junction (at 168.402 95.758) (diameter 1.016) (color 0 0 0 0))
-  (junction (at 138.43 141.478) (diameter 1.016) (color 0 0 0 0))
-  (junction (at 67.818 99.314) (diameter 1.016) (color 0 0 0 0))
-  (junction (at 116.332 95.758) (diameter 1.016) (color 0 0 0 0))
+  (junction (at 127.762 47.244) (diameter 1.016) (color 0 0 0 0)
+  )
+  (junction (at 185.42 141.478) (diameter 1.016) (color 0 0 0 0)
+  )
+  (junction (at 213.106 141.478) (diameter 1.016) (color 0 0 0 0)
+  )
+  (junction (at 78.994 117.856) (diameter 1.016) (color 0 0 0 0)
+  )
+  (junction (at 49.53 103.124) (diameter 1.016) (color 0 0 0 0)
+  )
+  (junction (at 147.32 95.758) (diameter 1.016) (color 0 0 0 0)
+  )
+  (junction (at 79.502 76.454) (diameter 1.016) (color 0 0 0 0)
+  )
+  (junction (at 232.41 23.876) (diameter 1.016) (color 0 0 0 0)
+  )
+  (junction (at 194.31 23.876) (diameter 1.016) (color 0 0 0 0)
+  )
+  (junction (at 138.43 141.478) (diameter 1.016) (color 0 0 0 0)
+  )
+  (junction (at 67.818 106.934) (diameter 1.016) (color 0 0 0 0)
+  )
+  (junction (at 194.31 141.478) (diameter 1.016) (color 0 0 0 0)
+  )
+  (junction (at 219.71 141.478) (diameter 1.016) (color 0 0 0 0)
+  )
+  (junction (at 78.994 47.498) (diameter 1.016) (color 0 0 0 0)
+  )
+  (junction (at 138.43 39.116) (diameter 1.016) (color 0 0 0 0)
+  )
+  (junction (at 178.816 74.93) (diameter 1.016) (color 0 0 0 0)
+  )
+  (junction (at 232.41 141.478) (diameter 1.016) (color 0 0 0 0)
+  )
+  (junction (at 178.816 63.754) (diameter 1.016) (color 0 0 0 0)
+  )
+  (junction (at 236.982 81.026) (diameter 1.016) (color 0 0 0 0)
+  )
+  (junction (at 168.402 81.026) (diameter 1.016) (color 0 0 0 0)
+  )
+  (junction (at 84.328 47.498) (diameter 1.016) (color 0 0 0 0)
+  )
+  (junction (at 78.994 141.478) (diameter 1.016) (color 0 0 0 0)
+  )
+  (junction (at 116.332 95.758) (diameter 1.016) (color 0 0 0 0)
+  )
+  (junction (at 116.332 23.876) (diameter 1.016) (color 0 0 0 0)
+  )
+  (junction (at 92.964 76.454) (diameter 1.016) (color 0 0 0 0)
+  )
+  (junction (at 116.332 58.166) (diameter 1.016) (color 0 0 0 0)
+  )
+  (junction (at 147.32 81.026) (diameter 1.016) (color 0 0 0 0)
+  )
+  (junction (at 227.33 81.026) (diameter 1.016) (color 0 0 0 0)
+  )
+  (junction (at 56.642 83.312) (diameter 1.016) (color 0 0 0 0)
+  )
+  (junction (at 240.03 23.876) (diameter 0) (color 0 0 0 0)
+  )
+  (junction (at 203.2 130.048) (diameter 1.016) (color 0 0 0 0)
+  )
+  (junction (at 67.818 64.77) (diameter 1.016) (color 0 0 0 0)
+  )
+  (junction (at 67.818 99.314) (diameter 1.016) (color 0 0 0 0)
+  )
+  (junction (at 168.402 95.758) (diameter 1.016) (color 0 0 0 0)
+  )
+  (junction (at 219.71 23.876) (diameter 1.016) (color 0 0 0 0)
+  )
+  (junction (at 203.2 35.814) (diameter 1.016) (color 0 0 0 0)
+  )
+  (junction (at 138.43 55.626) (diameter 1.016) (color 0 0 0 0)
+  )
+  (junction (at 78.994 23.876) (diameter 1.016) (color 0 0 0 0)
+  )
+  (junction (at 186.944 23.876) (diameter 1.016) (color 0 0 0 0)
+  )
+  (junction (at 92.71 141.478) (diameter 1.016) (color 0 0 0 0)
+  )
+  (junction (at 138.43 23.876) (diameter 1.016) (color 0 0 0 0)
+  )
+  (junction (at 178.816 141.478) (diameter 1.016) (color 0 0 0 0)
+  )
+  (junction (at 178.816 123.952) (diameter 1.016) (color 0 0 0 0)
+  )
+  (junction (at 92.71 23.876) (diameter 1.016) (color 0 0 0 0)
+  )
+  (junction (at 240.03 23.9261) (diameter 0) (color 0 0 0 0)
+  )
+  (junction (at 219.71 95.758) (diameter 1.016) (color 0 0 0 0)
+  )
+  (junction (at 92.71 124.46) (diameter 1.016) (color 0 0 0 0)
+  )
+  (junction (at 138.43 113.792) (diameter 1.016) (color 0 0 0 0)
+  )
+  (junction (at 178.816 107.188) (diameter 1.016) (color 0 0 0 0)
+  )
+  (junction (at 92.71 40.894) (diameter 1.016) (color 0 0 0 0)
+  )
+  (junction (at 67.818 57.15) (diameter 1.016) (color 0 0 0 0)
+  )
+  (junction (at 42.672 73.914) (diameter 1.016) (color 0 0 0 0)
+  )
+  (junction (at 213.106 23.876) (diameter 1.016) (color 0 0 0 0)
+  )
+  (junction (at 241.3 141.4597) (diameter 0) (color 0 0 0 0)
+  )
+  (junction (at 178.816 23.876) (diameter 1.016) (color 0 0 0 0)
+  )
   (wire (pts (xy 92.964 76.454) (xy 102.87 76.454))
     (stroke (width 0) (type solid) (color 0 0 0 0))
@@
     (effects (font (size 1.27 1.27)) (justify left bottom))
   )
-  (text "R27 : Vishay Dale 1W (CMF60560R00JKR6) or good low ppm resistor."
-    (at 93.98 173.99 0)
+  (text "R27 : Use good low noise and low ppm 1W resistor." (at 93.98 177.8 0)
     (effects (font (size 1.27 1.27)) (justify left bottom))
   )
@@
     (effects (font (size 1.27 1.27)) (justify left bottom))
   )
-  (text "Resistors 1W and 2W  : Vishay PR01 and PR02 (except R27)."
-    (at 93.98 177.8 0)
-    (effects (font (size 1.27 1.27)) (justify left bottom))
-  )
