File: Q17-Mini-1.2/Q17-Mini KiCad source/Q17-Mini.kicad_sch (KiCad schematic)
At the start: 87 parts, among them J1 Input, J2-1 SPK+, J2-2 SPK-, J3-1 V+, J3-2 GND, J3-3 V-, Q1 IRF610, Q10 KSA992, Q11 ZVP2106A, Q12 BD139, Q13 IRF610, Q14 IRF9610, Q15 FQA46N15, Q16 FQA36P15, Q2 KSA992, Q3 KSC1845, Q4 IRF9610, Q5 FQP3P20, Q6 FQP3N30, Q7 KSC1845, Q8 ZVN4206AV, Q9 ZVP2106A, U1 OPA1641

Commit message: Update Q17-Mini.kicad_sch
Parts:
- R22: value 100 -> STRAP
Other:
- note added: "C17 : 100nF MKP capacitor FKP3C031004C00JSSD or MKP1F031004B00KI00."
- note added: "C3, C6 : ELna Silmic II 100uF 16v"
- note added: "Q15 : FQA46N15"
- note added: "Q16 : FQA36P15"
- note removed: "C17 : 1uF MKP capacitor FKP3C031004C00JSSD or MKP1F031004B00KI00."
- note removed: "C3, C5 : ELna Silmic II 100uF 16v"
- note removed: "Q15 : FQA46N15 or IRF610"
- note removed: "Q16 : FQA36P15 or IRF9610"
- title: Q17-Mini Amplifier -> Q17-Mini 1.2 serie Amplifier
Changed lines of the file:
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@@
   (paper "A4")
   (title_block
-    (title "Q17-Mini Amplifier")
-    (date "2022-03-06")
-    (rev "1.3")
+    (title "Q17-Mini 1.2 serie Amplifier")
+    (date "2022-07-22")
+    (rev "1.3.3")
     (company "by eng. Tiberiu Vicol")
     (comment 1 "Modified by Stef for the Q17-Mini project")
@@
     (effects (font (size 1.27 1.27)) (justify left bottom))
   )
-  (text "C3, C5 : ELna Silmic II 100uF 16v" (at 59.69 179.07 0)
+  (text "C3, C6 : ELna Silmic II 100uF 16v" (at 59.69 179.07 0)
     (effects (font (size 1.27 1.27)) (justify left bottom))
   )
@@
     (effects (font (size 1.27 1.27)) (justify left bottom))
   )
-  (text "Q15 : FQA46N15 or IRF610" (at 13.97 194.31 0)
+  (text "Q15 : FQA46N15" (at 13.97 194.31 0)
     (effects (font (size 1.27 1.27)) (justify left bottom))
   )
@@
     (effects (font (size 1.27 1.27)) (justify left bottom))
   )
-  (text "C17 : 1uF MKP capacitor FKP3C031004C00JSSD or MKP1F031004B00KI00."
+  (text "C17 : 100nF MKP capacitor FKP3C031004C00JSSD or MKP1F031004B00KI00."
     (at 96.52 189.23 0)
     (effects (font (size 1.27 1.27)) (justify left bottom))
@@
     (effects (font (size 1.27 1.27)) (justify left bottom))
   )
-  (text "Q16 : FQA36P15 or IRF9610" (at 13.97 196.85 0)
+  (text "Q16 : FQA36P15" (at 13.97 196.85 0)
     (effects (font (size 1.27 1.27)) (justify left bottom))
   )
@@
     (in_bom yes) (on_board yes)
     (property "Reference" "R22" (id 0) (at 55.88 71.12 90))
-    (property "Value" "100" (id 1) (at 55.88 76.2 90))
+    (property "Value" "STRAP" (id 1) (at 55.88 76.2 90))
     (property "Footprint" "Resistor_THT:R_Axial_DIN0207_L6.3mm_D2.5mm_P10.16mm_Horizontal" (id 2) (at 55.88 75.438 90)
       (effects (font (size 1.27 1.27)) hide)
@@
     )
     (path "/bd791790-787e-4e23-9dad-9c957ce708c4"
-      (reference "R22") (unit 1) (value "100") (footprint "Resistor_THT:R_Axial_DIN0207_L6.3mm_D2.5mm_P10.16mm_Horizontal")
+      (reference "R22") (unit 1) (value "STRAP") (footprint "Resistor_THT:R_Axial_DIN0207_L6.3mm_D2.5mm_P10.16mm_Horizontal")
     )
     (path "/ee7cc794-8b46-4e6d-a64c-3ff4ac2fc69d"
