File: Q17-Mini 1.2.1/KiCad source/Q17-Mini.kicad_pcb (KiCad board)
At the start: 2 copper layers, 95 x 75 mm, 93 parts, among them J1 Input, J2-1 SPK+, J2-2 SPK-, J3-1 V+, J3-2 GND, J3-3 V-, Q1 IRF610, Q10 KSA992, Q11 ZVP2106A, Q12 BD139, Q13 IRF610, Q14 IRF9610, Q15 FQA46N15, Q16 FQA36P15, Q2 KSA992, Q3 KSC1845, Q4 IRF9610, Q5 FQP3P20, Q6 FQP3N30, Q7 KSC1845, Q8 ZVN4206AV, Q9 ZVP2106A, U1 OPA1641, U1' OPA1641

Commit message: Update diagram to 1.3.6
R29/R30 updated to 10k.
Parts:
- R29, R30: value 100R -> 10k
Changed lines of the file:
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@@
     (descr "Resistor, Axial_DIN0207 series, Axial, Horizontal, pin pitch=10.16mm, 0.25W = 1/4W, length*diameter=6.3*2.5mm^2, http://cdn-reichelt.de/documents/datenblatt/B400/1_4W%23YAG.pdf")
     (tags "Resistor Axial_DIN0207 series Axial Horizontal pin pitch 10.16mm 0.25W = 1/4W length 6.3mm diameter 2.5mm")
-    (property "Part#" "MRS25000C1000FC100")
+    (property "Part#" "MRS25000C1002FCT00")
     (property "Sheetfile" "Q17-Mini.kicad_sch")
     (property "Sheetname" "")
@@
       (effects (font (size 1 1) (thickness 0.15)))
     )
-    (fp_text value "100R" (at 5.08 2.37 90) (layer "F.Fab")
+    (fp_text value "10k" (at 5.08 2.37 90) (layer "F.Fab")
       (effects (font (size 1 1) (thickness 0.15)))
     )
@@
     (descr "Resistor, Axial_DIN0207 series, Axial, Horizontal, pin pitch=10.16mm, 0.25W = 1/4W, length*diameter=6.3*2.5mm^2, http://cdn-reichelt.de/documents/datenblatt/B400/1_4W%23YAG.pdf")
     (tags "Resistor Axial_DIN0207 series Axial Horizontal pin pitch 10.16mm 0.25W = 1/4W length 6.3mm diameter 2.5mm")
-    (property "Part#" "MRS25000C1000FC100")
+    (property "Part#" "MRS25000C1002FCT00")
     (property "Sheetfile" "Q17-Mini.kicad_sch")
     (property "Sheetname" "")
@@
       (effects (font (size 1 1) (thickness 0.15)))
     )
-    (fp_text value "100R" (at 5.08 2.37 90) (layer "F.Fab")
-      (effects (font (size 1 1) (thickness 0.15)))
-    )
+    (fp_text value "10k" (at 5.08 2.37 90) (layer "F.Fab")
+      (effects (font (size 1 1) (thickness 0.15)))
+    )

Commit message: Update Q17-Mini 1.2.1
Updated schematic.
Parts:
- R2, R21: value 5k6/1W -> 10k/1W
- R32: value 10R -> STRAP
Changed lines of the file:
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@@
       (effects (font (size 1 1) (thickness 0.15)))
     )
-    (fp_text value "10R" (at 5.08 2.37) (layer "F.Fab")
+    (fp_text value "STRAP" (at 5.08 2.37) (layer "F.Fab")
       (effects (font (size 1 1) (thickness 0.15)))
     )
@@
     (descr "Resistor, Axial_DIN0207 series, Axial, Horizontal, pin pitch=10.16mm, 0.25W = 1/4W, length*diameter=6.3*2.5mm^2, http://cdn-reichelt.de/documents/datenblatt/B400/1_4W%23YAG.pdf")
     (tags "Resistor Axial_DIN0207 series Axial Horizontal pin pitch 10.16mm 0.25W = 1/4W length 6.3mm diameter 2.5mm")
-    (property "Part#" "PR01000105601JR500")
+    (property "Part#" "PR01000101002JR500")
     (property "Sheetfile" "Q17-Mini.kicad_sch")
     (property "Sheetname" "")
@@
       (effects (font (size 1 1) (thickness 0.15)))
     )
-    (fp_text value "5k6/1W" (at 5.08 2.37) (layer "F.Fab")
+    (fp_text value "10k/1W" (at 5.08 2.37) (layer "F.Fab")
       (effects (font (size 1 1) (thickness 0.15)))
     )
@@
     (descr "Resistor, Axial_DIN0207 series, Axial, Horizontal, pin pitch=10.16mm, 0.25W = 1/4W, length*diameter=6.3*2.5mm^2, http://cdn-reichelt.de/documents/datenblatt/B400/1_4W%23YAG.pdf")
     (tags "Resistor Axial_DIN0207 series Axial Horizontal pin pitch 10.16mm 0.25W = 1/4W length 6.3mm diameter 2.5mm")
-    (property "Part#" "PR01000105601JR500")
+    (property "Part#" "PR01000101002JR500")
     (property "Sheetfile" "Q17-Mini.kicad_sch")
     (property "Sheetname" "")
@@
       (effects (font (size 1 1) (thickness 0.15)))
     )
-    (fp_text value "5k6/1W" (at 5.08 2.37 -90) (layer "F.Fab")
-      (effects (font (size 1 1) (thickness 0.15)))
-    )
+    (fp_text value "10k/1W" (at 5.08 2.37 -90) (layer "F.Fab")
+      (effects (font (size 1 1) (thickness 0.15)))
+    )
