File: Q17-TURBO 1.0/KiCad source/Q17-TURBO.kicad_pcb (KiCad board)
At the start: 2 copper layers, 190 x 75 mm, 107 parts, among them J1 INPUT, J2 SPK+, J3 DC, Q1 IRF610, Q10 KSA992, Q11 ZVP2106A, Q12 BD139, Q13 IRF610, Q14 IRF9610, Q15 FQA46N15, Q16 FQA36P15, Q17 FQA46N15, Q18 FQA36P15, Q2 KSA992, Q3 KSC1845, Q4 IRF9610, Q5 FQP3P20, Q6 FQP3N30, Q7 KSC1845, Q8 ZVN4206AV, Q9 ZVP2106A, U1 OPA1641, U1' OPA1641

Commit message: Update Q17-TURBO 1.0
Parts:
- C3, C6: value 100uF/16V -> 47uF/25v
Changed lines of the file:
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@@
   (title_block
     (title "Q17-TURBO (P2)")
-    (date "2022-09-09")
+    (date "2022-09-10")
     (rev "1.0")
     (company "PCB design by Stef")
@@
     (descr "CP, Radial series, Radial, pin pitch=5.00mm, , diameter=10mm, Electrolytic Capacitor")
     (tags "CP Radial series Radial pin pitch 5.00mm  diameter 10mm Electrolytic Capacitor")
-    (property "Part#" "RFS-16V101MH3#5")
+    (property "Part#" "Nichicon Muse UKZ1E470MPM")
     (property "Sheetfile" "Q17-TURBO.kicad_sch")
     (property "Sheetname" "")
@@
       (effects (font (size 1 1) (thickness 0.15)))
     )
-    (fp_text value "100uF/16V" (at 2.5 6.25 -90) (layer "F.Fab")
+    (fp_text value "47uF/25v" (at 2.5 6.25 -90) (layer "F.Fab")
       (effects (font (size 1 1) (thickness 0.15)))
     )
@@
     (descr "CP, Radial series, Radial, pin pitch=5.00mm, , diameter=10mm, Electrolytic Capacitor")
     (tags "CP Radial series Radial pin pitch 5.00mm  diameter 10mm Electrolytic Capacitor")
-    (property "Part#" "RFS-16V101MH3#5")
+    (property "Part#" "Nichicon Muse UKZ1E470MPM")
     (property "Sheetfile" "Q17-TURBO.kicad_sch")
     (property "Sheetname" "")
@@
       (effects (font (size 1 1) (thickness 0.15)))
     )
-    (fp_text value "100uF/16V" (at 2.5 6.25 90) (layer "F.Fab")
-      (effects (font (size 1 1) (thickness 0.15)))
-    )
+    (fp_text value "47uF/25v" (at 2.5 6.25 90) (layer "F.Fab")
+      (effects (font (size 1 1) (thickness 0.15)))
+    )

Commit message: Update Q17-TURBO 1.0 project
Parts:
- U1: value OPA1641 -> OPA1611
Changed lines of the file:
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@@
     (descr "SOIC, 8 Pin (JEDEC MS-012AA, https://www.analog.com/media/en/package-pcb-resources/package/pkg_pdf/soic_narrow-r/r_8.pdf), generated with kicad-footprint-generator ipc_gullwing_generator.py")
     (tags "SOIC SO")
-    (property "Part#" "OPA1641AID")
+    (property "Part#" "OPA1611AID")
     (property "Sheetfile" "Q17-TURBO.kicad_sch")
     (property "Sheetname" "")
@@
       (effects (font (size 1 1) (thickness 0.15)) (justify mirror))
     )
-    (fp_text value "OPA1641" (at 0 -3.4) (layer "B.Fab")
+    (fp_text value "OPA1611" (at 0 -3.4) (layer "B.Fab")
       (effects (font (size 1 1) (thickness 0.15)) (justify mirror))
     )
@@
     (effects (font (size 1 1) (thickness 0.15)))
   )
-  (gr_text "*" (at 62.6472 100.75) (layer "F.SilkS")
-    (effects (font (size 1 1) (thickness 0.15)))
-  )
+  (gr_text "*" (at 57.7472 123.05) (layer "F.SilkS")
+    (effects (font (size 1 1) (thickness 0.15)))
+  )

Commit message: Update Q17-TURBO 1.0 project
Parts:
- moved C8 16.4 mm to (81.6, 132.9), turned to -90 degrees
- moved D3 3.28 mm to (94.0, 133.9)
- moved Q1 3.28 mm to (87.6, 75.8)
- moved Q4 3.28 mm to (92.7, 141.2)
- moved R19 3.28 mm to (95.3, 83.9)
- moved R40 3.28 mm to (85.1, 79.7)
- moved R41 3.28 mm to (95.3, 137.7)
- moved R20 2.61 mm to (95.3, 130.2)
- moved D2 2.30 mm to (80.9, 83.6)
- moved C9 0.32 mm to (78.6, 91.3)
Routing:
- net Net-(C8-Pad2): track 28.2 -> 19.2 mm
- net Net-(C12-Pad2): track 115.4 -> 106.9 mm
- net Net-(C11-Pad2): track 132.0 -> 125.3 mm
- net Net-(C5-Pad2): track 53.0 -> 59.4 mm
- net Net-(C3-Pad1): track 65.9 -> 69.1 mm
- net Net-(C9-Pad2): track 49.0 -> 47.5 mm
- net Net-(Q3-Pad1): track 5.52 -> 6.55 mm
- net Net-(Q4-Pad1): track 4.60 -> 5.38 mm
- net Net-(Q2-Pad1): track 6.86 -> 7.57 mm
- net GND: vias 83 -> 75
Other:
- board text added: "M3"
