File: Q17-TURBO 1.0/KiCad source/Q17-TURBO.kicad_pcb (KiCad board)
At the start: 2 copper layers, 190 x 75 mm, 107 parts, among them J1 INPUT, J2 SPK+, J3 DC, Q1 IRF610, Q10 KSA992, Q11 ZVP2106A, Q12 BD139, Q13 IRF610, Q14 IRF9610, Q15 FQA46N15, Q16 FQA36P15, Q17 FQA46N15, Q18 FQA36P15, Q2 KSA992, Q3 KSC1845, Q4 IRF9610, Q5 FQP3P20, Q6 FQP3N30, Q7 KSC1845, Q8 ZVN4206AV, Q9 ZVP2106A, U1 OPA1611, U1' OPA1641

Commit message: Update Q17-TURBO 1.0 diagram
Parts:
- R29, R30: value 10k -> 100R
Changed lines of the file:
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@@
   (title_block
     (title "Q17-TURBO (P2)")
-    (date "2022-09-11")
+    (date "2022-09-14")
     (rev "1.0")
     (company "PCB design by Stef")
@@
     (descr "Resistor, Axial_DIN0207 series, Axial, Horizontal, pin pitch=10.16mm, 0.25W = 1/4W, length*diameter=6.3*2.5mm^2, http://cdn-reichelt.de/documents/datenblatt/B400/1_4W%23YAG.pdf")
     (tags "Resistor Axial_DIN0207 series Axial Horizontal pin pitch 10.16mm 0.25W = 1/4W length 6.3mm diameter 2.5mm")
-    (property "Part#" "MRS25000C1009FCT00")
+    (property "Part#" "MRS25000C1000FC100")
     (property "Sheetfile" "Q17-TURBO.kicad_sch")
     (property "Sheetname" "")
@@
       (effects (font (size 1 1) (thickness 0.15)))
     )
-    (fp_text value "10k" (at 5.08 0) (layer "F.SilkS") hide
+    (fp_text value "100R" (at 5.08 0) (layer "F.SilkS") hide
       (effects (font (size 1 1) (thickness 0.15)))
     )
@@
     (descr "Resistor, Axial_DIN0207 series, Axial, Horizontal, pin pitch=10.16mm, 0.25W = 1/4W, length*diameter=6.3*2.5mm^2, http://cdn-reichelt.de/documents/datenblatt/B400/1_4W%23YAG.pdf")
     (tags "Resistor Axial_DIN0207 series Axial Horizontal pin pitch 10.16mm 0.25W = 1/4W length 6.3mm diameter 2.5mm")
-    (property "Part#" "MRS25000C1009FCT00")
+    (property "Part#" "MRS25000C1000FC100")
     (property "Sheetfile" "Q17-TURBO.kicad_sch")
     (property "Sheetname" "")
@@
       (effects (font (size 1 1) (thickness 0.15)))
     )
-    (fp_text value "10k" (at 5.08 0) (layer "F.SilkS") hide
+    (fp_text value "100R" (at 5.08 0) (layer "F.SilkS") hide
       (effects (font (size 1 1) (thickness 0.15)))
     )
