File: Q17-TURBO 1.0/KiCad source/Q17-TURBO.kicad_sch (KiCad schematic)
At the start: 100 parts, among them J1 INPUT, J2 SPK+, J3 DC, Q1 IRF610, Q10 KSA992, Q11 ZVP2106A, Q12 BD139, Q13 IRF610, Q14 IRF9610, Q15 FQA46N15, Q16 FQA36P15, Q17 FQA46N15, Q18 FQA36P15, Q2 KSA992, Q3 KSC1845, Q4 IRF9610, Q5 FQP3P20, Q6 FQP3N30, Q7 KSC1845, Q8 ZVN4206AV, Q9 ZVP2106A, U1 OPA1641

Commit message: Update Q17-TURBO 1.0
Parts:
- C3, C6: value 100uF/16V -> 47uF/25v; Part# RFS-16V101MH3#5 -> Nichicon Muse UKZ1E470MPM
Changed lines of the file:
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@@
   (title_block
     (title "Q17-TURBO (P2) Amplifier")
-    (date "2022-09-09")
+    (date "2022-09-10")
     (rev "1.0")
     (company "by eng. Tiberiu Vicol")
@@
     (in_bom yes) (on_board yes)
     (property "Reference" "C6" (id 0) (at 54.1221 105.363 90))
-    (property "Value" "100uF/16V" (id 1) (at 56.134 112.776 90))
+    (property "Value" "47uF/25v" (id 1) (at 56.134 112.776 90))
     (property "Footprint" "Capacitor_THT:CP_Radial_D10.0mm_P5.00mm" (id 2) (at 60.96 106.9848 0)
       (effects (font (size 1.27 1.27)) hide)
@@
       (effects (font (size 1.27 1.27)) hide)
     )
-    (property "Part#" "RFS-16V101MH3#5" (id 4) (at 57.15 107.95 90)
+    (property "Part#" "Nichicon Muse UKZ1E470MPM" (id 4) (at 57.15 107.95 90)
       (effects (font (size 1.27 1.27)) hide)
     )
@@
     (in_bom yes) (on_board yes)
     (property "Reference" "C3" (id 0) (at 57.404 50.8 90))
-    (property "Value" "100uF/16V" (id 1) (at 57.404 53.0987 90))
+    (property "Value" "47uF/25v" (id 1) (at 57.404 53.0987 90))
     (property "Footprint" "Capacitor_THT:CP_Radial_D10.0mm_P5.00mm" (id 2) (at 53.34 58.1152 0)
       (effects (font (size 1.27 1.27)) hide)
@@
       (effects (font (size 1.27 1.27)) hide)
     )
-    (property "Part#" "RFS-16V101MH3#5" (id 4) (at 57.15 57.15 90)
+    (property "Part#" "Nichicon Muse UKZ1E470MPM" (id 4) (at 57.15 57.15 90)
       (effects (font (size 1.27 1.27)) hide)
     )
@@
     )
     (path "/f9e8c33b-6fda-41be-bb30-ce5c13715e36"
-      (reference "C3") (unit 1) (value "100uF/16V") (footprint "Capacitor_THT:CP_Radial_D10.0mm_P5.00mm")
+      (reference "C3") (unit 1) (value "47uF/25v") (footprint "Capacitor_THT:CP_Radial_D10.0mm_P5.00mm")
     )
     (path "/0c730a87-391f-4174-a498-479612b6c1cd"
@@
     )
     (path "/553e7843-c1ff-4dc6-ae3e-d89ae303f31a"
-      (reference "C6") (unit 1) (value "100uF/16V") (footprint "Capacitor_THT:CP_Radial_D10.0mm_P5.00mm")
+      (reference "C6") (unit 1) (value "47uF/25v") (footprint "Capacitor_THT:CP_Radial_D10.0mm_P5.00mm")
     )
     (path "/a9f732ba-8393-4274-8287-5fa363a75518"

Commit message: Update Q17-TURBO 1.0 project
Parts:
- U1: value OPA1641 -> OPA1611; Part# OPA1641AID -> OPA1611AID
Changed lines of the file:
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@@
       (effects (font (size 1.27 1.27)) (justify left))
     )
-    (property "Value" "OPA1641" (id 1) (at 66.04 71.12 0)
+    (property "Value" "OPA1611" (id 1) (at 66.04 71.12 0)
       (effects (font (size 1.27 1.27)) (justify left))
     )
@@
       (effects (font (size 1.27 1.27)) hide)
     )
-    (property "Part#" "OPA1641AID" (id 4) (at 66.04 76.2 0)
+    (property "Part#" "OPA1611AID" (id 4) (at 66.04 76.2 0)
       (effects (font (size 1.27 1.27)) hide)
     )
@@
     )
     (path "/92051f0d-a1e9-4769-b77b-885c48e9c81e"
-      (reference "U1") (unit 1) (value "OPA1641") (footprint "Package_SO:SOIC-8_3.9x4.9mm_P1.27mm")
-    )
-  )
+      (reference "U1") (unit 1) (value "OPA1611") (footprint "Package_SO:SOIC-8_3.9x4.9mm_P1.27mm")
+    )
+  )

Commit message: Update Q17-TURBO 1.0 project
Other:
- note added: "C3, C6 : Nichicon UKZ1E470MPM"
- note removed: "C3, C6 : ELna Silmic II 100uF 16v"
Changed lines of the file:
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@@
+    (effects (font (size 1.27 1.27)) (justify left bottom))
+  )
+  (text "C3, C6 : Nichicon UKZ1E470MPM" (at 59.69 179.07 0)
     (effects (font (size 1.27 1.27)) (justify left bottom))
   )
@@
     (effects (font (size 1.27 1.27)) (justify left bottom))
   )
-  (text "C3, C6 : ELna Silmic II 100uF 16v" (at 59.69 179.07 0)
-    (effects (font (size 1.27 1.27)) (justify left bottom))
-  )

Commit message: Update Q17-TURBO 1.0 diagram
Parts:
- R29, R30: value 10k -> 100R; Part# MRS25000C1009FCT00 -> MRS25000C1000FC100
Changed lines of the file:
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@@
   (title_block
     (title "Q17-TURBO (P2) Amplifier")
-    (date "2022-09-11")
-    (rev "1.0")
+    (date "2022-09-14")
+    (rev "1.0.1")
     (company "by eng. Tiberiu Vicol")
     (comment 1 "Modified by Stef for the Q17-TURBO project")
@@
       (effects (font (size 1.27 1.27)) (justify left))
     )
-    (property "Value" "10k" (id 1) (at 199.898 31.629 0)
+    (property "Value" "100R" (id 1) (at 199.898 31.629 0)
       (effects (font (size 1.27 1.27)) (justify left))
     )
@@
       (effects (font (size 1.27 1.27)) hide)
     )
-    (property "Part#" "MRS25000C1009FCT00" (id 4) (at 198.12 30.48 0)
+    (property "Part#" "MRS25000C1000FC100" (id 4) (at 198.12 30.48 0)
       (effects (font (size 1.27 1.27)) hide)
     )
@@
       (effects (font (size 1.27 1.27)) (justify left))
     )
-    (property "Value" "10k" (id 1) (at 199.4559 135.9102 0)
+    (property "Value" "100R" (id 1) (at 199.4559 135.9102 0)
       (effects (font (size 1.27 1.27)) (justify left))
     )
@@
       (effects (font (size 1.27 1.27)) hide)
     )
-    (property "Part#" "MRS25000C1009FCT00" (id 4) (at 198.12 134.62 0)
+    (property "Part#" "MRS25000C1000FC100" (id 4) (at 198.12 134.62 0)
       (effects (font (size 1.27 1.27)) hide)
     )
@@
     )
     (path "/6a502bca-5c03-4909-9915-ce87906e504a"
-      (reference "R29") (unit 1) (value "10k") (footprint "Resistor_THT:R_Axial_DIN0207_L6.3mm_D2.5mm_P10.16mm_Horizontal")
+      (reference "R29") (unit 1) (value "100R") (footprint "Resistor_THT:R_Axial_DIN0207_L6.3mm_D2.5mm_P10.16mm_Horizontal")
     )
     (path "/860cc2f6-176f-4935-b38a-f52437fa5513"
-      (reference "R30") (unit 1) (value "10k") (footprint "Resistor_THT:R_Axial_DIN0207_L6.3mm_D2.5mm_P10.16mm_Horizontal")
+      (reference "R30") (unit 1) (value "100R") (footprint "Resistor_THT:R_Axial_DIN0207_L6.3mm_D2.5mm_P10.16mm_Horizontal")
     )
     (path "/0b38258b-fc2c-4616-935a-ea7f37c299ab"

Commit message: Update schematics
Other:
- note added: "+13,99v"
- note added: "+17,44v"
- note added: "+48v"
- note added: "-14,32v"
- note added: "-48v"
- note added: "0,605v"
- note added: "0,774v"
- note added: "POWER 53vDC max 60v"
- note removed: "POWER 58vDC max 60v"
Changed lines of the file:
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@@
   (title_block
     (title "Q17-TURBO (P2) Amplifier")
-    (date "2022-09-14")
-    (rev "1.0.1")
+    (date "2023-02-18")
+    (rev "1.0.2")
     (company "by eng. Tiberiu Vicol")
     (comment 1 "Modified by Stef for the Q17-TURBO project")
@@
     (effects (font (size 1.27 1.27)) (justify left bottom))
   )
+  (text "+13,99v" (at 64.77 68.58 0)
+    (effects (font (size 1.27 1.27) italic) (justify left bottom))
+  )
   (text "Vz15v" (at 176.53 36.83 0)
     (effects (font (size 1.27 1.27)) (justify left bottom))
   )
+  (text "+48v" (at 181.61 22.86 0)
+    (effects (font (size 1.27 1.27) italic) (justify left bottom))
+  )
   (text "R27 : 560R 1W 1% Ohmite WNB560FET or Vishay CMF60560R00JKR6"
     (at 96.52 168.91 0)
@@
     (effects (font (size 1.27 1.27)) (justify left bottom))
   )
+  (text "0,774v" (at 107.9362 32.4403 90)
+    (effects (font (size 1.27 1.27) italic) (justify left bottom))
+  )
   (text "C17 : 100nF capacitor FKP3C031004C00JSSD or MKT1822410255."
     (at 96.52 186.69 0)
@@
     (effects (font (size 1.27 1.27)) (justify left bottom))
   )
+  (text "-48v" (at 180.34 144.78 0)
+    (effects (font (size 1.27 1.27) italic) (justify left bottom))
+  )
   (text "Remember to take off the resistors of 1W and more from the PCB when you solder them."
     (at 177.8 165.1 0)
@@
     (effects (font (size 1.27 1.27)) (justify left bottom))
   )
+  (text "0,605v" (at 165.6154 136.5264 90)
+    (effects (font (size 1.27 1.27) italic) (justify left bottom))
+  )
   (text "C2 : Non polar capacitor Nichicon Muse UES1A101MPM."
     (at 96.52 179.07 0)
@@
     (effects (font (size 1.27 1.27)) (justify left bottom))
   )
-  (text "POWER 58vDC\nmax 60v" (at 270.51 76.2 0)
+  (text "POWER 53vDC\nmax 60v" (at 270.51 76.2 0)
     (effects (font (size 1.27 1.27)) (justify left bottom))
   )
@@
     (effects (font (size 1.27 1.27)) (justify left bottom))
   )
+  (text "+17,44v" (at 97.79 62.23 0)
+    (effects (font (size 1.27 1.27) italic) (justify left bottom))
+  )
   (text "Measure across R13 for class A stage bias (60mA)." (at 13.97 30.48 0)
     (effects (font (size 1.27 1.27)) (justify left bottom))
@@
     (effects (font (size 1.27 1.27)) (justify left bottom))
   )
+  (text "-14,32v" (at 64.77 82.55 0)
+    (effects (font (size 1.27 1.27) italic) (justify left bottom))
+  )
   (text "optional" (at 233.68 133.35 0)
     (effects (font (size 1.27 1.27)) (justify left bottom))
@@
   (symbol (lib_id "Device:C") (at 101.6 34.29 0) (unit 1)
     (in_bom yes) (on_board yes)
-    (property "Reference" "C29" (id 0) (at 102.87 31.75 0)
+    (property "Reference" "C29" (id 0) (at 96.52 31.75 0)
       (effects (font (size 1.27 1.27)) (justify left))
     )
