File: Q17-Mini 1.3/KiCad source/Q17-Mini.kicad_pcb (KiCad board)
At the start: 2 copper layers, 95 x 75 mm, 93 parts, among them J1 Input, J2-1 SPK+, J2-2 SPK-, J3-1 V+, J3-2 GND, J3-3 V-, Q1 IRF610, Q10 KSA992, Q11 ZVP2106A, Q12 BD139, Q13 IRF610, Q14 IRF9610, Q15 FQA46N15, Q16 FQA36P15, Q2 KSA992, Q3 KSC1845, Q4 IRF9610, Q5 FQP3P20, Q6 FQP3N30, Q7 KSC1845, Q8 ZVN4206AV, Q9 ZVP2106A, U1 OPA1641, U1' OPA1641

Commit message: Update diagram for Q17-Mini 1.3
Parts:
- R1: value 2.7k -> 2k7
- R29, R30: value 100R -> 10k
Changed lines of the file:
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@@
   (title_block
     (title "Q17-Mini, the Quad405 reborn")
-    (date "2022-08-25")
+    (date "2022-08-29")
     (rev "1.3")
     (company "PCB design by Stef")
@@
     (descr "Resistor, Axial_DIN0207 series, Axial, Horizontal, pin pitch=10.16mm, 0.25W = 1/4W, length*diameter=6.3*2.5mm^2, http://cdn-reichelt.de/documents/datenblatt/B400/1_4W%23YAG.pdf")
     (tags "Resistor Axial_DIN0207 series Axial Horizontal pin pitch 10.16mm 0.25W = 1/4W length 6.3mm diameter 2.5mm")
-    (property "Part#" "MRS25000C1000FC100")
+    (property "Part#" "MRS25000C1002FCT00")
     (property "Sheetfile" "Q17-Mini.kicad_sch")
     (property "Sheetname" "")
@@
       (effects (font (size 1 1) (thickness 0.15)))
     )
-    (fp_text value "100R" (at 5.08 2.37 90) (layer "F.Fab")
+    (fp_text value "10k" (at 5.08 2.37 90) (layer "F.Fab")
       (effects (font (size 1 1) (thickness 0.15)))
     )
@@
     (descr "Resistor, Axial_DIN0207 series, Axial, Horizontal, pin pitch=10.16mm, 0.25W = 1/4W, length*diameter=6.3*2.5mm^2, http://cdn-reichelt.de/documents/datenblatt/B400/1_4W%23YAG.pdf")
     (tags "Resistor Axial_DIN0207 series Axial Horizontal pin pitch 10.16mm 0.25W = 1/4W length 6.3mm diameter 2.5mm")
-    (property "Part#" "MRS25000C1000FC100")
+    (property "Part#" "MRS25000C1002FCT00")
     (property "Sheetfile" "Q17-Mini.kicad_sch")
     (property "Sheetname" "")
@@
       (effects (font (size 1 1) (thickness 0.15)))
     )
-    (fp_text value "100R" (at 5.08 2.37 90) (layer "F.Fab")
+    (fp_text value "10k" (at 5.08 2.37 90) (layer "F.Fab")
       (effects (font (size 1 1) (thickness 0.15)))
     )
@@
       (effects (font (size 1 1) (thickness 0.15)))
     )
-    (fp_text value "2.7k" (at 5.08 2.37) (layer "F.Fab")
+    (fp_text value "2k7" (at 5.08 2.37) (layer "F.Fab")
       (effects (font (size 1 1) (thickness 0.15)))
     )

Commit message: Update Input_connector_mix_ footprint files
Parts:
- J1: value Input -> INPUT
Changed lines of the file:
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@@
   (title_block
     (title "Q17-Mini, the Quad405 reborn")
-    (date "2022-08-29")
+    (date "2022-09-01")
     (rev "1.3")
     (company "PCB design by Stef")
@@
     (descr "Terminal Block Phoenix PT-1,5-2-5.0-H, 2 pins, pitch 5mm, size 10x9mm^2, drill diamater 1.3mm, pad diameter 2.6mm, see http://www.mouser.com/ds/2/324/ItemDetail_1935161-922578.pdf, script-generated using https://github.com/pointhi/kicad-footprint-generator/scripts/TerminalBlock_Phoenix")
     (tags "THT Terminal Block Phoenix PT-1,5-2-5.0-H pitch 5mm size 10x9mm^2 drill 1.3mm pad 2.6mm")
-    (property "Part#" "Terminal Block KF128 5mm 2P")
+    (property "Part#" "Terminal Block KF127 5mm 2P")
     (property "Sheetfile" "Q17-Mini.kicad_sch")
     (property "Sheetname" "")
@@
       (effects (font (size 1 1) (thickness 0.15)))
     )
-    (fp_text value "Input" (at 2.3622 -5.4356 -90) (layer "F.Fab")
+    (fp_text value "INPUT" (at 2.3622 -5.4356 -90) (layer "F.Fab")
       (effects (font (size 1 1) (thickness 0.15)))
     )

Commit message: Upgraded Q17-Mini 1.3
Parts:
- C3, C6: value 100uF/16V -> 47uF/25v
- U1: value OPA1641 -> OPA1611
Changed lines of the file:
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@@
   (title_block
     (title "Q17-Mini, the Quad405 reborn")
-    (date "2022-09-07")
+    (date "2022-09-11")
     (rev "1.3")
     (company "PCB design by Stef")
@@
     (descr "CP, Radial series, Radial, pin pitch=5.00mm, , diameter=10mm, Electrolytic Capacitor")
     (tags "CP Radial series Radial pin pitch 5.00mm  diameter 10mm Electrolytic Capacitor")
-    (property "Part#" "RFS-16V101MH3#5")
+    (property "Part#" "Nichicon Muse UKZ1E470MPM")
     (property "Sheetfile" "Q17-Mini.kicad_sch")
     (property "Sheetname" "")
@@
       (effects (font (size 1 1) (thickness 0.15)))
     )
-    (fp_text value "100uF/16V" (at 2.5 6.25 90) (layer "F.Fab")
+    (fp_text value "47uF/25v" (at 2.5 6.25 90) (layer "F.Fab")
       (effects (font (size 1 1) (thickness 0.15)))
     )
@@
     (descr "CP, Radial series, Radial, pin pitch=5.00mm, , diameter=10mm, Electrolytic Capacitor")
     (tags "CP Radial series Radial pin pitch 5.00mm  diameter 10mm Electrolytic Capacitor")
-    (property "Part#" "RFS-16V101MH3#5")
+    (property "Part#" "Nichicon Muse UKZ1E470MPM")
     (property "Sheetfile" "Q17-Mini.kicad_sch")
     (property "Sheetname" "")
@@
       (effects (font (size 1 1) (thickness 0.15)))
     )
-    (fp_text value "100uF/16V" (at 2.5 6.25 90) (layer "F.Fab")
+    (fp_text value "47uF/25v" (at 2.5 6.25 90) (layer "F.Fab")
       (effects (font (size 1 1) (thickness 0.15)))
     )
@@
     (descr "SOIC, 8 Pin (JEDEC MS-012AA, https://www.analog.com/media/en/package-pcb-resources/package/pkg_pdf/soic_narrow-r/r_8.pdf), generated with kicad-footprint-generator ipc_gullwing_generator.py")
     (tags "SOIC SO")
-    (property "Part#" "OPA1641AID")
+    (property "Part#" "OPA1611AID")
     (property "Sheetfile" "Q17-Mini.kicad_sch")
     (property "Sheetname" "")
@@
       (effects (font (size 1 1) (thickness 0.15)) (justify mirror))
     )
-    (fp_text value "OPA1641" (at 0 -3.4) (layer "B.Fab")
+    (fp_text value "OPA1611" (at 0 -3.4) (layer "B.Fab")
       (effects (font (size 1 1) (thickness 0.15)) (justify mirror))
     )

Commit message: Update diagram for Q17-Mini 1.3
Changed R29/R30 to 100R.
Parts:
- R29, R30: value 10k -> 100R
Changed lines of the file:
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@@
     (descr "Resistor, Axial_DIN0207 series, Axial, Horizontal, pin pitch=10.16mm, 0.25W = 1/4W, length*diameter=6.3*2.5mm^2, http://cdn-reichelt.de/documents/datenblatt/B400/1_4W%23YAG.pdf")
     (tags "Resistor Axial_DIN0207 series Axial Horizontal pin pitch 10.16mm 0.25W = 1/4W length 6.3mm diameter 2.5mm")
-    (property "Part#" "MRS25000C1002FCT00")
+    (property "Part#" "MRS25000C1000FC100")
     (property "Sheetfile" "Q17-Mini.kicad_sch")
     (property "Sheetname" "")
@@
       (effects (font (size 1 1) (thickness 0.15)))
     )
-    (fp_text value "10k" (at 5.08 2.37 90) (layer "F.Fab")
+    (fp_text value "100R" (at 5.08 2.37 90) (layer "F.Fab")
       (effects (font (size 1 1) (thickness 0.15)))
     )
@@
     (descr "Resistor, Axial_DIN0207 series, Axial, Horizontal, pin pitch=10.16mm, 0.25W = 1/4W, length*diameter=6.3*2.5mm^2, http://cdn-reichelt.de/documents/datenblatt/B400/1_4W%23YAG.pdf")
     (tags "Resistor Axial_DIN0207 series Axial Horizontal pin pitch 10.16mm 0.25W = 1/4W length 6.3mm diameter 2.5mm")
-    (property "Part#" "MRS25000C1002FCT00")
+    (property "Part#" "MRS25000C1000FC100")
     (property "Sheetfile" "Q17-Mini.kicad_sch")
     (property "Sheetname" "")
@@
       (effects (font (size 1 1) (thickness 0.15)))
     )
-    (fp_text value "10k" (at 5.08 2.37 90) (layer "F.Fab")
-      (effects (font (size 1 1) (thickness 0.15)))
-    )
+    (fp_text value "100R" (at 5.08 2.37 90) (layer "F.Fab")
+      (effects (font (size 1 1) (thickness 0.15)))
+    )
