File: Q17-PSU-1.0.1/KiCad source/Q17-PSU.kicad_sch (KiCad schematic)
At the start: 31 parts, among them J1-1 AC1-1, J1-2 AC1-2, J1-3 AC2-1, J1-4 AC2-2, J2-1 V+, J2-2 V+, J2-3 GNDPWR, J2-4 GNDPWR, J2-5 GNDPWR, J2-6 V-, J2-7 V-

Commit message: Update Q17-PSU files
Parts:
- C1: Mouser R76QF21005050J -> 80-PHE426MK5100JR05; Part# 80-R76QF21005050J -> PHE426MK5100JR05
- C2: Mouser 80-R76QF21005050J -> 80-PHE426MK5100JR05; Part# R76QF21005050J -> PHE426MK5100JR05
Changed lines of the file:
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@@
   (title_block
     (title "Q17 Power Supply Universal")
-    (date "2023-08-21")
+    (date "2023-08-22")
     (rev "1.0.1")
     (company "by stef")
@@
       (effects (font (size 1.27 1.27)) hide)
     )
-    (property "Datasheet" "https://www.mouser.fr/datasheet/2/212/1/KEM_F3034_R76-1103045.pdf" (at 83.82 77.47 0)
-      (effects (font (size 1.27 1.27)) hide)
-    )
-    (property "Part#" "80-R76QF21005050J" (at 83.82 77.47 0)
-      (effects (font (size 1.27 1.27)) hide)
-    )
-    (property "Mouser" "R76QF21005050J" (at 83.82 77.47 0)
+    (property "Datasheet" "https://www.mouser.fr/datasheet/2/212/F3294_PHE426-1101077.pdf" (at 83.82 77.47 0)
+      (effects (font (size 1.27 1.27)) hide)
+    )
+    (property "Part#" "PHE426MK5100JR05" (at 83.82 77.47 0)
+      (effects (font (size 1.27 1.27)) hide)
+    )
+    (property "Mouser" "80-PHE426MK5100JR05" (at 83.82 77.47 0)
       (effects (font (size 1.27 1.27)) hide)
     )
@@
       (effects (font (size 1.27 1.27)) hide)
     )
-    (property "Datasheet" "https://www.mouser.fr/datasheet/2/212/1/KEM_F3034_R76-1103045.pdf" (at 83.82 106.68 0)
-      (effects (font (size 1.27 1.27)) hide)
-    )
-    (property "Part#" "R76QF21005050J" (at 83.82 106.68 0)
-      (effects (font (size 1.27 1.27)) hide)
-    )
-    (property "Mouser" "80-R76QF21005050J" (at 83.82 106.68 0)
-      (effects (font (size 1.27 1.27)) hide)
-    )
+    (property "Datasheet" "https://www.mouser.fr/datasheet/2/212/F3294_PHE426-1101077.pdf" (at 83.82 106.68 0)
+      (effects (font (size 1.27 1.27)) hide)
+    )
+    (property "Part#" "PHE426MK5100JR05" (at 83.82 106.68 0)
+      (effects (font (size 1.27 1.27)) hide)
+    )
+    (property "Mouser" "80-PHE426MK5100JR05" (at 83.82 106.68 0)
+      (effects (font (size 1.27 1.27)) hide)
+    )

Commit message: Update files for BOM.
Parts:
- C1, C2: Mouser 80-PHE426MK5100JR05 -> 505-MKP1G021002C00KF; Part# PHE426MK5100JR05 -> MKP1G021002C00KF00
Changed lines of the file:
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@@
       (effects (font (size 1.27 1.27)) hide)
     )
-    (property "Datasheet" "https://www.mouser.fr/datasheet/2/212/F3294_PHE426-1101077.pdf" (at 83.82 77.47 0)
+    (property "Datasheet" "https://www.mouser.fr/datasheet/2/440/e_WIMA_MKP_10-1139811.pdf" (at 83.82 77.47 0)
       (effects (font (size 1.27 1.27)) hide)
     )
-    (property "Part#" "PHE426MK5100JR05" (at 83.82 77.47 0)
+    (property "Part#" "MKP1G021002C00KF00" (at 83.82 77.47 0)
       (effects (font (size 1.27 1.27)) hide)
     )
-    (property "Mouser" "80-PHE426MK5100JR05" (at 83.82 77.47 0)
+    (property "Mouser" "505-MKP1G021002C00KF" (at 83.82 77.47 0)
       (effects (font (size 1.27 1.27)) hide)
     )
@@
       (effects (font (size 1.27 1.27)) hide)
     )
-    (property "Datasheet" "https://www.mouser.fr/datasheet/2/212/F3294_PHE426-1101077.pdf" (at 83.82 106.68 0)
+    (property "Datasheet" "https://www.mouser.fr/datasheet/2/440/e_WIMA_MKP_10-1139811.pdf" (at 83.82 106.68 0)
       (effects (font (size 1.27 1.27)) hide)
     )
-    (property "Part#" "PHE426MK5100JR05" (at 83.82 106.68 0)
+    (property "Part#" "MKP1G021002C00KF00" (at 83.82 106.68 0)
       (effects (font (size 1.27 1.27)) hide)
     )
-    (property "Mouser" "80-PHE426MK5100JR05" (at 83.82 106.68 0)
+    (property "Mouser" "505-MKP1G021002C00KF" (at 83.82 106.68 0)
       (effects (font (size 1.27 1.27)) hide)
     )
