File: Q17-PSU-1.0.3/KiCad source/Q17-PSU.kicad_sch (KiCad schematic)
At the start: 31 parts, among them J1-1 AC1-1, J1-2 AC1-2, J1-3 AC2-1, J1-4 AC2-2, J2-1 V+, J2-2 V+, J2-3 GNDPWR, J2-4 GNDPWR, J2-5 GNDPWR, J2-6 V-, J2-7 V-

Commit message: Q17-PSU version 1.0.3
Parts:
- C1, C2: footprint Capacitor_THT:C_Rect_L10.0mm_W4.0mm_P7.50mm_MKS4 -> Capacitor_THT:C_Disc_D6.0mm_W4.4mm_P5.00mm
Other:
- note added: "Others film capacitors : MKP X2"
- note removed: "Others capacitors : MKP X2"
Changed lines of the file:
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@@
     (effects (font (size 1.27 1.27)) (justify left bottom))
   )
-  (text "C1, C2 : 10nF 100V NPO (COG)" (at 83.82 170.18 0)
+  (text "C1, C2 : 10nF 100V NPO (COG)" (at 15.24 157.48 0)
     (effects (font (size 1.27 1.27)) (justify left bottom))
   )
@@
     (effects (font (size 1.27 1.27)) (justify left bottom))
   )
-  (text "Others capacitors : MKP X2" (at 83.82 173.99 0)
+  (text "Others film capacitors : MKP X2" (at 15.24 161.29 0)
     (effects (font (size 1.27 1.27)) (justify left bottom))
   )
@@
       (effects (font (size 1.27 1.27)) (justify left))
     )
-    (property "Footprint" "Capacitor_THT:C_Rect_L10.0mm_W4.0mm_P7.50mm_MKS4" (at 84.7852 81.28 0)
+    (property "Footprint" "Capacitor_THT:C_Disc_D6.0mm_W4.4mm_P5.00mm" (at 84.7852 81.28 0)
       (effects (font (size 1.27 1.27)) hide)
     )
@@
       (effects (font (size 1.27 1.27)) (justify left))
     )
-    (property "Footprint" "Capacitor_THT:C_Rect_L10.0mm_W4.0mm_P7.50mm_MKS4" (at 84.7852 110.49 0)
+    (property "Footprint" "Capacitor_THT:C_Disc_D6.0mm_W4.4mm_P5.00mm" (at 84.7852 110.49 0)
       (effects (font (size 1.27 1.27)) hide)
     )
