File: Q17-PSU-1.0.3/KiCad source/Q17-PSU.kicad_pcb (KiCad board)
At the start: 2 copper layers, 102 x 102 mm, 36 parts, among them J1-1 AC1-1, J1-2 AC1-2, J1-3 AC2-1, J1-4 AC2-2, J2-1 V+, J2-2 V+, J2-3 GNDPWR, J2-4 GNDPWR, J2-5 GNDPWR, J2-6 V-, J2-7 V-

Commit message: Q17-PSU version 1.0.3
Parts:
- C1, C2: footprint Capacitor_THT:C_Rect_L10.0mm_W4.0mm_P7.50mm_MKS4 -> Capacitor_THT:C_Disc_D6.0mm_W4.4mm_P5.00mm
- moved C1 1.25 mm to (106.0, 69.3)
- moved C2 1.25 mm to (106.0, 107.6)
Routing:
- net Net-(J1-2-Pin_1): track 51.6 -> 60.2 mm
- net Net-(J1-4-Pin_1): track 41.8 -> 43.8 mm
Other:
- board text added: "Q17-PSU 1.0.3"
- board text removed: "Q17-PSU 1.0.2"

Commit message: Update Q17-PSU 1.0.3
Routing:
- net Net-(C4-Pad2): track 9.93 -> 11.1 mm
