File: Q17-PSU-1.0.4/KiCad source/Q17-PSU.kicad_pcb (KiCad board)
At the start: 2 copper layers, 102 x 102 mm, 36 parts, among them J1-1 AC1-1, J1-2 AC1-2, J1-3 AC2-1, J1-4 AC2-2, J2-1 V+, J2-2 V+, J2-3 GNDPWR, J2-4 GNDPWR, J2-5 GNDPWR, J2-6 V-, J2-7 V-

Commit message: Q17-PSU v1.0.4
Routing:
- net Net-(J1-3-Pin_1): track 65.0 -> 55.9 mm
- net Net-(J1-2-Pin_1): track 60.2 -> 54.9 mm
- net Net-(J1-4-Pin_1): track 43.8 -> 40.1 mm
- net Net-(J1-1-Pin_1): track 53.4 -> 50.7 mm
Other:
- board text added: "Q17-PSU 1.0.4"
- board text removed: "Q17-PSU 1.0.3"
Changed lines of the file:
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@@
   (title_block
     (title "Q17 Power Supply")
-    (date "2023-08-30")
-    (rev "1.0.3")
+    (date "2023-09-06")
+    (rev "1.0.4")
     (company "by stef")
   )
@@
     (effects (font (size 1 1) (thickness 0.15)) (justify bottom))
   )
-  (gr_text "Q17-PSU 1.0.3" (at 104.902 79.248 270) (layer "F.SilkS")
+  (gr_text "Q17-PSU 1.0.4" (at 104.902 79.248 270) (layer "F.SilkS")
     (effects (font (size 2 2) (thickness 0.4) bold) (justify left bottom))
   )
@@
   (segment (start 100.71228 63.246) (end 100.71228 58.166) (width 3) (layer "F.Cu") (net 2))
   (arc (start 106.498328 69.032048) (mid 106.822751 69.248821) (end 107.205435 69.324941) (width 3) (layer "F.Cu") (net 2))
-  (segment (start 119.018447 50.907553) (end 124.567554 45.358446) (width 1) (layer "B.Cu") (net 2))
-  (segment (start 118.872 66.086893) (end 118.872 51.261107) (width 1) (layer "B.Cu") (net 2))
-  (segment (start 115.970447 69.195553) (end 118.725554 66.440446) (width 1) (layer "B.Cu") (net 2))
-  (segment (start 111.523059 69.342) (end 115.616893 69.342) (width 1) (layer "B.Cu") (net 2))
-  (segment (start 124.921107 45.212) (end 127.762 45.212) (width 1) (layer "B.Cu") (net 2))
-  (arc (start 118.725554 66.440446) (mid 118.83394 66.278234) (end 118.872 66.086893) (width 1) (layer "B.Cu") (net 2))
-  (arc (start 118.872 51.261107) (mid 118.91006 51.069765) (end 119.018447 50.907553) (width 1) (layer "B.Cu") (net 2))
-  (arc (start 115.616893 69.342) (mid 115.808235 69.30394) (end 115.970447 69.195553) (width 1) (layer "B.Cu") (net 2))
-  (arc (start 124.921107 45.212) (mid 124.729766 45.25006) (end 124.567554 45.358446) (width 1) (layer "B.Cu") (net 2))
+  (segment (start 111.523059 69.342) (end 118.325107 62.539952) (width 1) (layer "B.Cu") (net 2))
+  (segment (start 118.910893 51.269107) (end 124.675107 45.504893) (width 1) (layer "B.Cu") (net 2))
+  (segment (start 125.382214 45.212) (end 127.762 45.212) (width 1) (layer "B.Cu") (net 2))
+  (segment (start 118.618 61.832845) (end 118.618 51.976214) (width 1) (layer "B.Cu") (net 2))
+  (arc (start 124.675107 45.504893) (mid 124.99953 45.28812) (end 125.382214 45.212) (width 1) (layer "B.Cu") (net 2))
+  (arc (start 118.910893 51.269107) (mid 118.69412 51.59353) (end 118.618 51.976214) (width 1) (layer "B.Cu") (net 2))
+  (arc (start 118.325107 62.539952) (mid 118.54188 62.215529) (end 118.618 61.832845) (width 1) (layer "B.Cu") (net 2))
   (segment (start 106.630827 107.264547) (end 100.71228 101.346) (width 3) (layer "F.Cu") (net 3))
   (segment (start 100.71228 101.346) (end 100.71228 96.266) (width 3) (layer "F.Cu") (net 3))
   (segment (start 111.506 107.55744) (end 107.337934 107.55744) (width 3) (layer "F.Cu") (net 3))
   (arc (start 106.630827 107.264547) (mid 106.95525 107.48132) (end 107.337934 107.55744) (width 3) (layer "F.Cu") (net 3))
-  (segment (start 125.984 110.697107) (end 125.984 116.124893) (width 1) (layer "B.Cu") (net 3))
-  (segment (start 111.506 107.55744) (end 122.844333 107.55744) (width 1) (layer "B.Cu") (net 3))
-  (segment (start 131.064 121.619107) (end 131.064 135.428893) (width 1) (layer "B.Cu") (net 3))
-  (segment (start 126.130447 116.478447) (end 130.917554 121.265554) (width 1) (layer "B.Cu") (net 3))
-  (segment (start 130.917553 135.782447) (end 130.116683 136.583317) (width 1) (layer "B.Cu") (net 3))
-  (segment (start 123.197887 107.703887) (end 125.837554 110.343554) (width 1) (layer "B.Cu") (net 3))
-  (segment (start 129.76313 136.729763) (end 127.762 136.729763) (width 1) (layer "B.Cu") (net 3))
-  (arc (start 122.844333 107.55744) (mid 123.035675 107.5955) (end 123.197887 107.703887) (width 1) (layer "B.Cu") (net 3))
-  (arc (start 130.917554 121.265554) (mid 131.02594 121.427766) (end 131.064 121.619107) (width 1) (layer "B.Cu") (net 3))
-  (arc (start 125.984 116.124893) (mid 126.02206 116.316235) (end 126.130447 116.478447) (width 1) (layer "B.Cu") (net 3))
-  (arc (start 125.984 110.697107) (mid 125.94594 110.505766) (end 125.837554 110.343554) (width 1) (layer "B.Cu") (net 3))
-  (arc (start 130.116683 136.583317) (mid 129.954471 136.691703) (end 129.76313 136.729763) (width 1) (layer "B.Cu") (net 3))
-  (arc (start 130.917553 135.782447) (mid 131.02594 135.620235) (end 131.064 135.428893) (width 1) (layer "B.Cu") (net 3))
+  (segment (start 111.506 107.55744) (end 114.001226 107.55744) (width 1) (layer "B.Cu") (net 3))
+  (segment (start 114.708333 107.850333) (end 127.469107 120.611107) (width 1) (layer "B.Cu") (net 3))
+  (segment (start 127.762 121.318214) (end 127.762 136.729763) (width 1) (layer "B.Cu") (net 3))
+  (arc (start 127.469107 120.611107) (mid 127.68588 120.93553) (end 127.762 121.318214) (width 1) (layer "B.Cu") (net 3))
+  (arc (start 114.708333 107.850333) (mid 114.38391 107.63356) (end 114.001226 107.55744) (width 1) (layer "B.Cu") (net 3))
   (segment (start 100.728887 80.501393) (end 100.71228 80.518) (width 3) (layer "F.Cu") (net 4))
   (segment (start 106.04628 74.324941) (end 106.04628 76.699221) (width 1.5) (layer "F.Cu") (net 4))
@@
   (segment (start 111.506 76.824941) (end 104.819553 76.824941) (width 3) (layer "F.Cu") (net 4))
   (arc (start 104.112446 77.117834) (mid 104.436869 76.901061) (end 104.819553 76.824941) (width 3) (layer "F.Cu") (net 4))
-  (segment (start 123.698 53.594) (end 123.698 73.452893) (width 1) (layer "B.Cu") (net 4))
-  (segment (start 120.325952 76.824941) (end 111.506 76.824941) (width 1) (layer "B.Cu") (net 4))
-  (segment (start 123.551553 73.806447) (end 120.679505 76.678495) (width 1) (layer "B.Cu") (net 4))
-  (arc (start 123.698 73.452893) (mid 123.65994 73.644235) (end 123.551553 73.806447) (width 1) (layer "B.Cu") (net 4))
-  (arc (start 120.325952 76.824941) (mid 120.517293 76.786881) (end 120.679505 76.678495) (width 1) (layer "B.Cu") (net 4))
+  (segment (start 123.698 53.594) (end 123.698 64.218727) (width 1) (layer "B.Cu") (net 4))
+  (segment (start 123.405107 64.925834) (end 111.506 76.824941) (width 1) (layer "B.Cu") (net 4))
+  (arc (start 123.698 64.218727) (mid 123.62188 64.60141) (end 123.405107 64.925834) (width 1) (layer "B.Cu") (net 4))
   (segment (start 111.506 115.05744) (end 104.941054 115.05744) (width 3) (layer "F.Cu") (net 5))
   (segment (start 104.233947 115.350333) (end 100.71228 118.872) (width 3) (layer "F.Cu") (net 5))
@@
   (segment (start 106.04628 112.55744) (end 106.04628 114.92916) (width 1.5) (layer "F.Cu") (net 5))
   (arc (start 104.233947 115.350333) (mid 104.55837 115.13356) (end 104.941054 115.05744) (width 3) (layer "F.Cu") (net 5))
-  (segment (start 118.759887 115.203887) (end 119.995554 116.439554) (width 1) (layer "B.Cu") (net 5))
-  (segment (start 120.288447 126.638447) (end 122.027554 128.377554) (width 1) (layer "B.Cu") (net 5))
-  (segment (start 111.506 115.05744) (end 118.406333 115.05744) (width 1) (layer "B.Cu") (net 5))
-  (segment (start 122.381107 128.524) (end 123.698 128.524) (width 1) (layer "B.Cu") (net 5))
-  (segment (start 120.142 116.793107) (end 120.142 126.284893) (width 1) (layer "B.Cu") (net 5))
-  (arc (start 119.995554 116.439554) (mid 120.10394 116.601766) (end 120.142 116.793107) (width 1) (layer "B.Cu") (net 5))
-  (arc (start 118.406333 115.05744) (mid 118.597675 115.0955) (end 118.759887 115.203887) (width 1) (layer "B.Cu") (net 5))
-  (arc (start 122.381107 128.524) (mid 122.189766 128.48594) (end 122.027554 128.377554) (width 1) (layer "B.Cu") (net 5))
-  (arc (start 120.142 126.284893) (mid 120.18006 126.476235) (end 120.288447 126.638447) (width 1) (layer "B.Cu") (net 5))
+  (segment (start 111.506 115.05744) (end 113.373226 115.05744) (width 1) (layer "B.Cu") (net 5))
+  (segment (start 114.080333 115.350333) (end 123.405107 124.675107) (width 1) (layer "B.Cu") (net 5))
+  (segment (start 123.698 125.382214) (end 123.698 128.524) (width 1) (layer "B.Cu") (net 5))
+  (arc (start 123.405107 124.675107) (mid 123.62188 124.99953) (end 123.698 125.382214) (width 1) (layer "B.Cu") (net 5))
+  (arc (start 114.080333 115.350333) (mid 113.75591 115.13356) (end 113.373226 115.05744) (width 1) (layer "B.Cu") (net 5))
   (segment (start 172.866447 46.453833) (end 175.236834 44.083446) (width 1) (layer "F.Cu") (net 6))
   (segment (start 175.590387 43.937) (end 177.8 43.937) (width 1) (layer "F.Cu") (net 6))
