File: Q17-PSU-1.0.4/KiCad source/Q17-PSU.kicad_sch (KiCad schematic)
At the start: 31 parts, among them J1-1 AC1-1, J1-2 AC1-2, J1-3 AC2-1, J1-4 AC2-2, J2-1 V+, J2-2 V+, J2-3 GNDPWR, J2-4 GNDPWR, J2-5 GNDPWR, J2-6 V-, J2-7 V-

Commit message: Update PSU BOM
Parts:
- R6: Mouser PR01000101002JR500 -> 594-5073NW10K00J; Part# 594-5073NW10K00J -> PR01000101002JR500
Changed lines of the file:
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@@
       (effects (font (size 1.27 1.27)) hide)
     )
-    (property "Part#" "594-5073NW10K00J" (at 193.04 104.14 0)
+    (property "Part#" "PR01000101002JR500" (at 193.04 104.14 0)
       (effects (font (size 1.27 1.27)) hide)
     )
-    (property "Mouser" "PR01000101002JR500" (at 193.04 104.14 0)
+    (property "Mouser" "594-5073NW10K00J" (at 193.04 104.14 0)
       (effects (font (size 1.27 1.27)) hide)
     )
