File: Q17-SIGMA-PSU-1.1/KiCad source/Q17-SIGMA-PSU.kicad_pcb (KiCad board)
At the start: 2 copper layers, 130 x 75 mm, 84 parts, among them J1-1 V+ (IN), J1-2 GND, J1-3 V- (IN), J2-1 V+, J2-2 V+, J2-3 GND, J2-4 GND, J2-5 GND, J2-6 V-, J2-7 V-, Q1 BC548B, Q2 BC558B, Q3 BC548B, Q4 BC556B, Q5 BC546B, Q6 IRFZ24NPBF, Q7 IRF9Z34NPBF, Q8 IRFZ24NPBF, Q9 IRF9Z34NPBF, U1 ZHB6792TA, U2 ZHB6792TA

Commit message: Q17-SIGMA-PSU 1.1 update
Parts:
- U1, U2: footprint Package_TO_SOT_SMD:TSOT-23-8_HandSoldering -> Package_TO_SOT_SMD:SOT-223-8
- moved C12 25.6 mm to (142.8, 79.5), turned to 0 degrees
- moved C13 17.7 mm to (147.8, 117.3), turned to 180 degrees
- moved R19 16.2 mm to (161.3, 110.0), turned to 0 degrees
- moved R5 14.1 mm to (159.3, 88.1)
- moved CR4 7.64 mm to (138.9, 114.8), turned to 180 degrees
- moved CR1 7.62 mm to (132.1, 86.1), turned to 0 degrees
- moved C15 4.72 mm to (176.5, 106.4)
- moved C14 3.81 mm to (179.7, 86.4)
- moved U2 2.32 mm to (151.8, 106.5)
- moved CR3 1.61 mm to (170.7, 99.1)
- moved Q5 0.26 mm to (142.7, 113.0)
- moved U1 0.20 mm to (151.8, 91.8)
- renumbered REF** to PAD3
Routing:
- net Net-(CR4-K): track 97.8 -> 55.7 mm
- net Net-(Q4-B): track 32.3 -> 11.2 mm
- net /V- (OUT): track 19.2 -> 33.0 mm
- net Net-(Q5-B): track 32.1 -> 24.0 mm, vias 0 -> 1
- net Net-(CR1-K): track 7.91 -> 15.4 mm
- net Net-(U1-B1): track 3.76 -> 11.0 mm
- net Net-(U1-B3): track 28.6 -> 23.2 mm, vias 0 -> 1
- net Net-(U2-B2): track 6.51 -> 11.7 mm
- net Net-(CR2-A): track 7.84 -> 12.3 mm
- net /GND: track 53.1 -> 57.5 mm, vias 1 -> 0
- net Net-(C14-Pad1): track 29.7 -> 25.8 mm
- net Net-(Q3-B): track 28.0 -> 24.5 mm
- net Net-(U2-B4): track 34.3 -> 31.3 mm
- net Net-(U1-B2): track 46.6 -> 48.8 mm
- net Net-(Q3-C): track 36.3 -> 38.1 mm
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Other:
- board text added: "Q17-SIGMA-PSU 1.1"
- board text removed: "Q17-SIGMA-PSU 1.0"
