File: Q17-SIGMA-PSU-1.1/KiCad source/Q17-SIGMA-PSU.kicad_sch (KiCad schematic)
At the start: 80 parts, among them J1-1 V+ (IN), J1-2 GND, J1-3 V- (IN), J2-1 V+, J2-2 V+, J2-3 GND, J2-4 GND, J2-5 GND, J2-6 V-, J2-7 V-, Q1 BC548B, Q2 BC558B, Q3 BC548B, Q4 BC556B, Q5 BC546B, Q6 IRFZ24NPBF, Q7 IRF9Z34NPBF, Q8 IRFZ24NPBF, Q9 IRF9Z34NPBF, U1 ZHB6792TA, U2 ZHB6792TA

Commit message: Q17-SIGMA-PSU 1.1 update
Parts:
- U1, U2: footprint Package_TO_SOT_SMD:TSOT-23-8_HandSoldering -> Package_TO_SOT_SMD:SOT-223-8
Other:
- note added: "C1, C2, C16, C17 : 1uF 100V Wima MKP MKP1D041005G00KSSD (use MKP pulse caps)"
- note added: "C12, C13 : 3900pF 100V Kemet MMK5392J100J01L16.5TA18 or Kemet PHE426DJ4390JR05"
- note added: "C14, C15 : 220pF 100V Kemet C0G C315C221J1G"
- note added: "C5, C6, C7, C8, C11 : 100uF 80V Panasonic EEU-FS1K101 (low ESR, miniature)"
- note removed: "100uF = Panasonic EEU-FS1K101 (low ESR, miniature)"
- note removed: "1uF = Wima MKP MKP1D041005G00KSSD (use MKP pulse caps)"
- note removed: "220pF 100V = Kemet C0G C315C221J1G"
- note removed: "3900pF 100V = Kemet MMK5392J100J01L16.5TA18 or Kemet PHE426DJ4390JR05"
- note removed: "All capacitors rated for 80V/100V minimum."
Changed lines of the file:
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@@
 	(title_block
 		(title "Q17-SIGMA Power Supply")
-		(date "2024-04-20")
-		(rev "1.0.5")
+		(date "2024-04-22")
+		(rev "1.0.7")
 		(company "PCB and BOM by stef")
 		(comment 2 "Design and test by Moor")
@@
 		)
 	)
-	(text "All capacitors rated for 80V/100V minimum."
-		(exclude_from_sim no)
-		(at 14.732 156.21 0)
-		(effects
-			(font
-				(size 1.27 1.27)
-			)
-			(justify left)
-		)
-	)
-	(text "1uF = Wima MKP MKP1D041005G00KSSD (use MKP pulse caps)"
+	(text "C1, C2, C16, C17 : 1uF 100V Wima MKP MKP1D041005G00KSSD (use MKP pulse caps)"
 		(exclude_from_sim no)
 		(at 14.478 171.45 0)
@@
 		)
 	)
-	(text "100uF = Panasonic EEU-FS1K101 (low ESR, miniature)"
+	(text "C5, C6, C7, C8, C11 : 100uF 80V Panasonic EEU-FS1K101 (low ESR, miniature)"
 		(exclude_from_sim no)
 		(at 14.478 173.99 0)
@@
 		)
 	)
-	(text "3900pF 100V = Kemet MMK5392J100J01L16.5TA18 or Kemet PHE426DJ4390JR05"
+	(text "C12, C13 : 3900pF 100V Kemet MMK5392J100J01L16.5TA18 or Kemet PHE426DJ4390JR05"
 		(exclude_from_sim no)
 		(at 14.478 166.37 0)
@@
 	(text "Q7, Q9 : IRF9Z34NPBF or IRF9540NPBF"
 		(exclude_from_sim no)
-		(at 14.732 153.67 0)
+		(at 14.478 156.21 0)
 		(effects
 			(font
@@
 	(text "Q6, Q8 : IRFZ24NPBF or IRF530NPBF"
 		(exclude_from_sim no)
-		(at 14.732 151.13 0)
+		(at 14.478 153.67 0)
 		(effects
 			(font
@@
 		)
 	)
-	(text "220pF 100V = Kemet C0G C315C221J1G "
+	(text "C14, C15 : 220pF 100V Kemet C0G C315C221J1G "
 		(exclude_from_sim no)
 		(at 14.478 168.91 0)
@@
 			)
 		)
-		(property "Footprint" "Package_TO_SOT_SMD:TSOT-23-8_HandSoldering"
+		(property "Footprint" "Package_TO_SOT_SMD:SOT-223-8"
 			(at 157.48 40.64 0)
 			(effects
@@
 			)
 		)
-		(property "Footprint" "Package_TO_SOT_SMD:TSOT-23-8_HandSoldering"
+		(property "Footprint" "Package_TO_SOT_SMD:SOT-223-8"
 			(at 157.48 90.17 0)
 			(effects
