File: Q17-Mini-3.0/KiCad source/Q17-Mini.kicad_pcb (KiCad board)
At the start: 2 copper layers, 95 x 75 mm, 92 parts, among them J1 INPUT, J2-1 SPK+, J2-2 SPK-, J3-1 V+, J3-2 GND, J3-3 V-, Q1 IRF610, Q1' SI2328DS, Q10 KSA992, Q11 BS250P, Q111 BS250P, Q12 KSC1845, Q13 IRF610, Q14 IRF9610, Q15 FQA46N15, Q16 IXTQ36P15P, Q2 KSA992, Q3 KSC1845, Q4 IRF9610, Q4' SI2325DS, Q5 FQPF7P20, Q6 2SK3564, Q7 LSK170B, Q7' JFE150, Q8 DN2540, Q9 BS250P, U1 OPA1611, U1' OPA1611, U2 NDC7003P

Commit message: Update Q17-Mini to 3.0.4
Parts:
- added HBR: PinHeader_1x02_P2.54mm_Vertical, Connector_PinHeader_2.54mm:PinHeader_1x02_P2.54mm_Vertical, F.Cu at (146.0, 97.9)
- Q6: value 2SK3564 -> FQPF3N80C
- U1, U1': value OPA1611 -> OPA828
Routing:
- net GND: track 4.25 -> 23.4 mm
- net Net-(J2-1-Pin_1): track 33.5 -> 31.7 mm
Other:
- board text added: "HBR"
- board text added: "Q17-Mini 3.0.4"
- board text removed: "Q17-Mini 3.0.3"
